Commit message: remove everything but arms from kbot model and put it in roughly the right place

File: src/lerobot/teleoperators/vuer_vr/assets/kbot/robot.urdf (robot description, URDF)
Before this commit: robot kbotv2p0_nohands, 23 links, 22 joints
Links:
- removed link KB_D_501L_L_LEG_FOOT
- removed link KB_D_501R_R_LEG_FOOT
- removed link KC_D_102L_L_Hip_Yoke_Drive
- removed link KC_D_102R_R_Hip_Yoke_Drive
- removed link KC_D_301L_L_Femur_Lower_Drive
- removed link KC_D_301R_R_Femur_Lower_Drive
- removed link KC_D_401L_L_Shin_Drive
- removed link KC_D_401R_R_Shin_Drive
- removed link RS03_4
- removed link RS03_5
- removed link imu
- link Torso_Side_Right: geometry 
Joints:
- removed joint dof_left_ankle_02
- removed joint dof_left_hip_pitch_04
- removed joint dof_left_hip_roll_03
- removed joint dof_left_hip_yaw_03
- removed joint dof_left_knee_04
- removed joint dof_right_ankle_02
- removed joint dof_right_hip_pitch_04
- removed joint dof_right_hip_roll_03
- removed joint dof_right_hip_yaw_03
- removed joint dof_right_knee_04
- removed joint frame_imu_site

Commit message: modify urdf to have separate base link for left side kinematic chain

File: src/lerobot/teleoperators/vuer_vr/assets/kbot/robot.urdf (robot description, URDF)
Before this commit: robot kbotv2p0_nohands, 12 links, 11 joints
Links:
- added link Torso_Side_Left
- link Torso_Side_Right: mass 13.504988 -> None
Joints:
- added joint base_joint_left: type fixed, parent base, child Torso_Side_Left, origin xyz=0 -0.095 0 rpy=0 0 1.5708
- joint dof_left_shoulder_pitch_03: parent Torso_Side_Right -> Torso_Side_Left
